File: 4.Hardware/perfusion_placa_eagle/projects/Perfusion/perfusion_esquematico.brd (EAGLE design)
At the start: 100.3 x 100.3 mm, 13 parts

Commit message: [MOD] Fixes hardware
Parts:
- removed U$1: RELAY-2-SRD, diy-modules:RELAY-2-SRD
- added J4, J5, J6: (no value), SparkFun-Connectors:1X03
- added J7: (no value), SparkFun-Connectors:1X04_LONGPADS
- moved J2 89.2 mm to (56.6, 8.64), turned to 0 degrees
- moved J3 85.3 mm to (39.1, 8.64), turned to 0 degrees
- moved U$7 52.5 mm to (52.6, 31.5)
- moved U$8 42.2 mm to (70.4, 31.5), turned to 90 degrees
- moved U$2 36.1 mm to (43.4, 66.0)
- moved U$3 31.4 mm to (28.2, 38.9)
- moved PCB1 6.90 mm to (-44.5, 82.5)
- moved J1 2.18 mm to (22.6, 8.89)
- moved JUMPER 2.18 mm to (24.1, 18.8)
Connections:
- removed net GND.2: U$1.J2.3
- removed net RELAY_IN1: PCB1.P$15, U$1.J1.3
- removed net RELAY_IN2: PCB1.P$13, U$1.J1.2
- removed net VCC.2: U$1.J2.2
- new net DOUT_BAR: J7.2, PCB1.P$16
- new net HALL1: J4.3, PCB1.P$33
- new net HALL2: J5.3, PCB1.P$31
- new net HALL3: J6.3, PCB1.P$29
- new net SCK_BAR: J7.3, PCB1.P$18
- net RPI3_+3V: now also J4.2, J5.2, J6.2, J7.1
- net RPI3_+5V: no longer U$1.J1.1
- net RPI3_GND: now also J4.1, J5.1, J6.1, J7.4; no longer U$1.J1.4
- net SPI0_CS0: now also PCB1.P$11; no longer PCB1.P$24
- net SPI0_CS1: now also PCB1.P$7; no longer PCB1.P$26
Routing:
- net SPI0_CS0: track 66.3 -> 263.0 mm, vias 0 -> 2
- net HALL1: track 0.00 -> 130.8 mm
- net RELAY_IN1: track 123.3 -> 0.00 mm
- net SCK_BAR: track 0.00 -> 119.6 mm, vias 0 -> 2
- net HALL2: track 0.00 -> 118.3 mm
- net RELAY_IN2: track 113.1 -> 0.00 mm
- net HALL3: track 0.00 -> 107.4 mm
- net DOUT_BAR: track 0.00 -> 99.9 mm, vias 0 -> 6
- net RPI3_+3V: track 167.6 -> 265.8 mm, vias 2 -> 3
- net SPI0_CS1: track 77.9 -> 168.3 mm, vias 0 -> 3
- net SPI0_MOSI: track 263.1 -> 210.3 mm, vias 1 -> 3
- net RPI3_GND: track 356.5 -> 318.8 mm, vias 2 -> 3
- net RPI3_+5V: track 158.8 -> 123.1 mm, vias 0 -> 1
- net THERMO_CS3: track 90.0 -> 118.1 mm, vias 2 -> 4
- net I2C_SCL: track 66.6 -> 92.4 mm
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- added copper zone on layer 1, net RPI3_GND
- added copper zone on layer 16, net RPI3_GND
Other:
- board text added: "3.3V"
- board text added: "GND VIAS"
- board text added: "HALL_1"
- board text added: "HALL_2"
- board text added: "HALL_3"
- board text added: "OUT"
- board text added: "PRESSURE"
- board text added: "PUMP_1"
- board text added: "PUMP_2"
- board text added: "SCK"
- board text removed: "2 CHANNEL RELAY"
- board text removed: "BUZZER"
- board text removed: "DAC PUMP1"
- board text removed: "DAC PUMP2"
- board text removed: "PERFUSION V1.0 alejandrolucas@us.es +34 619939928 Dpto. FISICA APLICADA III"
- board text removed: "PUMP1"
- board text removed: "PUMP2"
