File: 4.Hardware/perfusion_placa_eagle/projects/Perfusion/perfusion_esquematico.sch (EAGLE design)
At the start: 13 parts

Commit message: [MOD] Fixes hardware
Parts:
- removed U$1: RELAY-2-SRD, diy-modules:RELAY-2-SRD
- added J4, J5, J6: (no value), SparkFun-Connectors:CONN_03
- added J7: (no value), SparkFun-Connectors:CONN_04LONGPADS
Connections:
- removed net RELAY_IN1: PCB1.GPIO22, U$1.IN1
- removed net RELAY_IN2: PCB1.GPIO27, U$1.IN2
- new net DOUT_BAR: J7.2, PCB1.GPIO23
- new net HALL1: J4.3, PCB1.GPIO13
- new net HALL2: J5.3, PCB1.GPIO6
- new net HALL3: J6.3, PCB1.GPIO5
- new net SCK_BAR: J7.3, PCB1.GPIO24
- net RPI3_+3V: now also J4.2, J5.2, J6.2, J7.1
- net RPI3_+5V: no longer U$1.VCC.1
- net RPI3_GND: now also J4.1, J5.1, J6.1, J7.4; no longer U$1.GND.1
- net SPI0_CS0: now also PCB1.GPIO17; no longer PCB1.GPIO8
- net SPI0_CS1: now also PCB1.GPIO4; no longer PCB1.GPIO7
Other:
- moved on the sheet: J1, J2, J3, JUMPER, U$2, U$3
